File: inzynierka/inzynierka.kicad_sch (KiCad schematic)
At the start: 33 parts, among them J1 OLED_128x32, J2 USB_C_Receptacle_USB2.0_16P, J3 con, Q1 DMP1045U, U1 CAT24C256, U2 USBLC6-2SC6, U3 TP4057, U4 DW01A, U5 dual nmos, U7 TPS63802DLAR

Commit message: Add files via upload
Connections:
- net GND: no longer C1.2, J3.2 (Pin_2), U4.6 (GND), U5.6 (S2), U5.7 (S2)
- net 5V renamed VBUS
- new net -BAT: C1.2, J3.2 (Pin_2), U4.6 (GND), U5.6 (S2), U5.7 (S2)
Other:
- note added: "MCU"

Commit message: Add files via upload
Parts:
- added C27: 0.1uF, Capacitor_SMD:C_0603_1608Metric, symbol Device:C
- added D4, D5, D6, D7: Diode, Diode_SMD:D_0603_1608Metric, symbol KEYBOARD:Placeholder_Diode
- added J5: Magnetic connector1, symbol Connector:Conn_01x04_Pin
- added J6: Magnetic connector2, symbol Connector:Conn_01x04_Pin
- added R16, R17: 4.7k, Resistor_SMD:R_0603_1608Metric, symbol Device:R
- added R19: 10k, Resistor_SMD:R_0603_1608Metric, symbol Device:R
- added S1, S2, S3, S4: Keyswitch, kbd:keyswitch_cherrymx_hotswap_1u, symbol KEYBOARD:Placeholder_Keyswitch
- added SW1: SW_Push, Button_Switch_SMD:SW_Push_1P1T_NO_CK_KMR2, symbol Switch:SW_Push
Connections:
- net +3.3V: now also R16.1, R17.1, R19.1
- net GND: now also C27.2, D4.1 (K), D5.1 (K), D6.1 (K), D7.1 (K), J5.4 (Pin_4), J6.4 (Pin_4), SW1.2
- net SCL: now also R17.2
- net SDA: now also R16.2
- net VBUS: now also J5.1 (Pin_1), J6.1 (Pin_1)
- new net: D6.2 (A), S3.2
- new net: D7.2 (A), S4.2
- new net: D5.2 (A), S2.2
- new net: D4.2 (A), S1.2
- new net RESET: C27.1, R19.2, SW1.1
- new net UARTRX: J5.2 (Pin_2), J6.3 (Pin_3)
- new net UARTTX: J5.3 (Pin_3), J6.2 (Pin_2)
- new net button1: S1.1
- new net button2: S2.1
- new net button3: S3.1
- new net button4: S4.1
Other:
- note added: "Button"
- note added: "KEYCAPS"
- note added: "Magnetic connectors"
- note added: "Reset button"
- note added: "i2c"
